File: Boards/MPPT/Mk5/MPPTMk5.kicad_pcb (KiCad board)
At the start: 4 copper layers, 49.7 x 54.6 mm, 62 parts, among them J1 Solar 1, J10 Conn_GND_Pin, J11 Conn_01x01_Pin, J12 LiPo, J13 LiPo, J2 Solar 2, J3 Solar 3, J4 LiPo, J5 LiPo, J6 Conn_01x07, J7 10kOhm Thermistor, J8 System, J9 USB_C_Receptacle_USB2.0, U1 BQ25672RQMR, U2 BQ34110PW, U3 BQ34110PW

Commit message: New files
use these :)
Parts:
- removed J12, J13, J5: LiPo, Connector_JST:JST_PH_S2B-PH-K_1x02_P2.00mm_Horizontal
- removed U1: BQ25672RQMR, BQ25672RQMR:IC_BQ25672RQMR
- removed U3: BQ34110PW, BQ34110:SOP65P640X120-14N
- added D2: LED, LED_SMD:LED_0402_1005Metric, F.Cu at (109.0, 53.2)
- added D3: LED, LED_SMD:LED_0402_1005Metric, F.Cu at (127.8, 67.1)
- added D4: LED, LED_SMD:LED_0402_1005Metric, F.Cu at (99.3, 70.0)
- added R14: 2.2kOhm, Resistor_SMD:R_0402_1005Metric, F.Cu at (99.2, 68.0)
- added R3: 2.2kOhm, Resistor_SMD:R_0402_1005Metric, F.Cu at (110.9, 53.2)
- added R4: 2.2kOhm, Resistor_SMD:R_0402_1005Metric, F.Cu at (127.8, 69.0)
- R2: value 6.04kOhm -> 8.2kOhm
- U2: value BQ34110PW -> BQ25798RQMR; footprint BQ34110:SOP65P640X120-14N -> BQ25798RQMR:IC_BQ25798RQMR
- moved U2 21.6 mm to (113.8, 77.3)
- moved J4 12.0 mm to (114.0, 50.7)
- moved J10 9.93 mm to (90.0, 84.9)
- moved J11 9.85 mm to (97.8, 91.0)
- moved TP1 4.63 mm to (111.8, 54.9)
- moved G*** 3.65 mm to (132.8, 58.5)
- moved TP2 2.05 mm to (114.3, 54.9)
Connections:
- C17 pad 1: Net-(C17-Pad1) -> Net-(J4-Pin_2)
- C18 pad 1: Net-(C17-Pad1) -> Net-(J4-Pin_2)
- R7 pad 2: Net-(C17-Pad1) -> Net-(J4-Pin_2)
- TP1 pad 1: Net-(C17-Pad1) -> Net-(J4-Pin_2)
- U2 pad 2: unconnected-(U2-ALERT1-Pad2) -> Net-(U2-VBUS-Pad2)
- U2 pad 3: unconnected-(U2-LEN-Pad3) -> Net-(U2-VBUS-Pad2)
- U2 pad 5: Net-(J13-Pin_2) -> unconnected-(U2-REGN-Pad5)
Routing:
- net Net-(J4-Pin_2): track 11.2 -> 47.3 mm, vias 0 -> 1
- net Net-(C17-Pad1): track 22.2 -> 0.00 mm, vias 2 -> 0
- net Net-(J12-Pin_2): track 11.1 -> 0.00 mm
- net GND: track 59.3 -> 66.5 mm, vias 22 -> 25
- net Net-(J11-Pin_1): track 10.9 -> 4.88 mm
- net Net-(D3-A): track 0.00 -> 0.95 mm
- net Net-(D4-A): track 0.00 -> 0.92 mm
- net Net-(D2-A): track 0.00 -> 0.92 mm
- net VBUS: track 75.5 -> 76.3 mm
- net SYS: track 18.3 -> 19.1 mm
- net unconnected-(J5-Pin_2-Pad2): track 0.54 -> 0.00 mm
- added copper zone on In2.Cu, net (none)
- removed copper zone on In2.Cu, net SYS
Other:
- board size 49.7 x 54.6 mm -> 49.7 x 50.4 mm
- board text added: "BMS 2S2P"
- board text added: "LiPo IN"
- board text removed: "2S2P"
- board text removed: "LiPo"
